Commit message: change neupan_controller to nav2_mppi_controller

File: Simulation/gazebo_sim/urdf/robot/plugins/gazebo_control_plugin.xacro (robot description, xacro)
@@ -40,4 +40,5 @@
                 <odometry_frame>odom</odometry_frame>
                 <robot_base_frame>base_footprint</robot_base_frame>
+                <odometry_topic>odom</odometry_topic>
                 <!-- 发布频率（单位Hz） -->
                 <publish_rate>100</publish_rate>

File: Simulation/gazebo_sim/urdf/robot/robot.urdf.xacro (robot description, xacro)
@@ -6,24 +6,23 @@
     <xacro:include filename="car_base.urdf.xacro" />
     <xacro:include filename="sensor/velodyne.urdf.xacro" />
-    <xacro:include filename="sensor/camera.urdf.xacro" />
+    <!-- <xacro:include filename="sensor/camera.urdf.xacro" /> -->
     <!-- <xacro:include filename="laser.urdf.xacro" /> -->
-    <joint name="camera2base_link" type="fixed">
+    <!-- <joint name="camera2base_link" type="fixed">
         <parent link="vehicle" />
         <child link="camera" />
         <origin xyz="0.2 0 0.12" rpy="0 0 0" />
         <axis xyz="0 0 0" />
-    </joint>
-    <xacro:VLP-16 parent="vehicle" name="velodyne" topic="/velodyne_points" hz="10"
-        min_range="0.55" samples="350" collision_range="0.56" organize_cloud="true" gpu="false"
-        min_angle="0" max_angle="3.14159" vmin_angle="${-7/180*PI}" vmax_angle="${52/180*PI}">
-        <origin xyz="0.0 0.2 ${car_height/2+0.02}" rpy="0 0 0" />
+    </joint> -->
+    <xacro:VLP-16 parent="lidar_holder" name="velodyne" topic="/velodyne_points" hz="10"
+        min_range="0.55" samples="350" collision_range="0.56" gpu="false"
+        min_angle="-3.14159" max_angle="3.14159" vmin_angle="${-7/180*PI}" vmax_angle="${52/180*PI}">
+        <origin xyz="0.0 0.0 ${holder_length/2}" rpy="0 0 0" />
     </xacro:VLP-16>
-    <xacro:VLP-16 parent="vehicle" name="velodyne2" topic="/velodyne_points2" hz="10"
-        min_range="0.55" samples="350" collision_range="0.56" organize_cloud="true" gpu="false"
+    <!-- <xacro:VLP-16 parent="vehicle" name="velodyne2" topic="/velodyne_points2" hz="10"
+        min_range="0.55" samples="350" collision_range="0.56" gpu="false"
         min_angle="-3.14159" max_angle="0" vmin_angle="${-7/180*PI}" vmax_angle="${52/180*PI}">
         <origin xyz="0.0 -0.2 ${car_height/2+0.02}" rpy="0 0 0" />
-    </xacro:VLP-16>
-    <xacro:include
-        filename="$(find gazebo_sim)/urdf/robot/plugins/gazebo_control_plugin.xacro" />
-    <xacro:base_mecanum_gazebo />
+    </xacro:VLP-16> -->
+    <xacro:include filename="$(find gazebo_sim)/urdf/robot/plugins/gazebo_control_plugin.xacro" />
+    <xacro:gazebo_control_plugin />
 </robot>

File: Simulation/velodyne_simulator/velodyne_description/urdf/VLP-16.urdf.xacro (robot description, xacro)
@@ -2,5 +2,5 @@
 <robot xmlns:xacro="http://www.ros.org/wiki/xacro" name="VLP-16">
   <xacro:property name="M_PI" value="3.1415926535897931"/>
-  <xacro:macro name="VLP-16" params="*origin parent:=base_link name:=velodyne topic:=/velodyne_points hz:=10 lasers:=16 samples:=1875 collision_range:=0.3 min_range:=0.9 max_range:=130.0 noise:=0.008 min_angle:=-${M_PI} max_angle:=${M_PI} gpu:=false">
+  <xacro:macro name="VLP-16" params="*origin parent:=base_link name:=velodyne topic:=/velodyne_points hz:=10 lasers:=16 samples:=1875 collision_range:=0.3 min_range:=0.9 max_range:=130.0 noise:=0.008 min_angle:=-${M_PI} max_angle:=${M_PI} gpu:=false vmin_angle:=-${M_PI} vmax_angle:=${M_PI}">
     <joint name="${name}_base_mount_joint" type="fixed">
       <xacro:insert_block name="origin"/>
@@ -71,7 +71,6 @@
                 <samples>${lasers}</samples>
                 <resolution>1</resolution>
-                <min_angle>-${15.0*M_PI/180.0}</min_angle>
-                <max_angle>
-                  ${15.0*M_PI/180.0}</max_angle>
+                <min_angle>${vmin_angle}</min_angle>
+                <max_angle>${vmax_angle}</max_angle>
               </vertical>
             </scan>
@@ -112,7 +111,6 @@
                 <samples>${lasers}</samples>
                 <resolution>1</resolution>
-                <min_angle>-${15.0*M_PI/180.0}</min_angle>
-                <max_angle>
-                  ${15.0*M_PI/180.0}</max_angle>
+                <min_angle>${vmin_angle}</min_angle>
+                <max_angle>${vmax_angle}</max_angle>
               </vertical>
             </scan>
