Commit message: launch with nodes[] failed

File: Simulation/gazebo_sim/urdf/robot/plugins/gazebo_control_plugin_prefix.xacro (robot description, xacro)
@@ -1,6 +1,5 @@
 <?xml version="1.0"?>
 <robot xmlns:xacro="http://www.ros.org/wiki/xacro">
-    <xacro:macro name="gazebo_control_plugin" params="hub_id:=''">
-        <xacro:property name="namespace_prefix" value="${hub_id + '/' if hub_id else ''}" />
+    <xacro:macro name="gazebo_control_plugin" params="namespace_prefix:=''">
         <!-- mu1静,mu2动，kp 刚度系数 kd 阻尼系数 -->
         <gazebo reference="${namespace_prefix}front_left_wheel">

File: Simulation/gazebo_sim/urdf/robot/property.xacro (robot description, xacro)
@@ -1,5 +1,5 @@
 <robot xmlns:xacro="http://www.ros.org/wiki/xacro" name="robot">
     <xacro:property name="hub_id" value="$(arg hub_id)" />
-    <xacro:property name="namespace_prefix" value="${hub_id + '/' if hub_id else ''}" />
+    <xacro:property name="namespace_prefix" value="${hub_id + '/'}" />
     <xacro:property name="ns" value="$(arg ns)/" />
     <!-- 惯性矩阵 -->

File: Simulation/gazebo_sim/urdf/robot/robot.urdf.xacro (robot description, xacro)
@@ -14,9 +14,9 @@
         <axis xyz="0 0 0" />
     </joint> -->
-    <xacro:VLP-16 hub_id="${hub_id}" parent="lidar_holder"  name="velodyne" topic="velodyne_points" hz="10"
+    <!-- <xacro:VLP-16 hub_id="${hub_id}" parent="lidar_holder"  name="velodyne" topic="velodyne_points" hz="10"
         min_range="0.55" samples="350" collision_range="0.56" gpu="false"
         min_angle="-3.14159" max_angle="3.14159" vmin_angle="${-7/180*PI}" vmax_angle="${52/180*PI}">
         <origin xyz="0.0 0.0 ${holder_length/2}" rpy="0 0 0" />
-    </xacro:VLP-16>
+    </xacro:VLP-16> -->
     <!-- <xacro:VLP-16 parent="vehicle" name="velodyne2" topic="/velodyne_points2" hz="10"
         min_range="0.55" samples="350" collision_range="0.56" gpu="false"
@@ -25,4 +25,4 @@
     </xacro:VLP-16> -->
     <xacro:include filename="$(find gazebo_sim)/urdf/robot/plugins/gazebo_control_plugin_prefix.xacro" />
-    <xacro:gazebo_control_plugin hub_id="${hub_id}" />
+    <xacro:gazebo_control_plugin namespace_prefix="${namespace_prefix}" />
 </robot>

File: Simulation/velodyne_simulator/velodyne_description/urdf/VLP-16.urdf.xacro (robot description, xacro)
@@ -20,10 +20,10 @@
       <visual>
         <geometry>
-          <mesh filename="package://velodyne_description/meshes/VLP16_base_1.dae" />
+          <mesh filename="file://$(find velodyne_description)/meshes/VLP16_base_1.dae"/>
         </geometry>
       </visual>
       <visual>
         <geometry>
-          <mesh filename="package://velodyne_description/meshes/VLP16_base_2.dae" />
+          <mesh filename="file://$(find velodyne_description)/meshes/VLP16_base_2.dae"/>
         </geometry>
       </visual>

Commit message: run successfully, navigation meeting bug

File: Simulation/gazebo_sim/urdf/robot/plugins/gazebo_control_plugin_prefix.xacro (robot description, xacro)
@@ -1,5 +1,5 @@
 <?xml version="1.0"?>
 <robot xmlns:xacro="http://www.ros.org/wiki/xacro">
-    <xacro:macro name="gazebo_control_plugin" params="namespace_prefix:=''">
+    <xacro:macro name="gazebo_control_plugin">
         <!-- mu1静,mu2动，kp 刚度系数 kd 阻尼系数 -->
         <gazebo reference="${namespace_prefix}front_left_wheel">
@@ -37,12 +37,16 @@
         <gazebo>
             <plugin name="planar_move_controller" filename="libgazebo_ros_planar_move.so">
-                <!-- 里程计和机器人基坐标系，添加命名空间前缀 -->
+                <!-- 里程计和机器人基坐标系，添加命名空间前缀，头两行在ros2中不支持 -->
+                <ros>
+                    <!-- <namespace>${robot_namespace}</namespace> -->
+                    <remapping>odom:=${namespace_prefix}odom</remapping>
+                    <remapping>cmd_vel:=${namespace_prefix}cmd_vel</remapping>
+                </ros>
                 <odometry_frame>${namespace_prefix}odom</odometry_frame>
                 <robot_base_frame>${namespace_prefix}base_footprint</robot_base_frame>
-                <odometry_topic>${namespace_prefix}odom</odometry_topic>
                 <!-- 发布频率（单位Hz） -->
-                <publish_rate>50</publish_rate>
+                <publish_rate>10</publish_rate>
                 <!-- 控制更新频率（可选，默认20Hz） -->
-                <update_rate>50</update_rate>
+                <update_rate>20</update_rate>
                 <!-- 是否发布里程计和TF（可选，默认true） -->
                 <publish_odom>true</publish_odom>

File: Simulation/gazebo_sim/urdf/robot/property.xacro (robot description, xacro)
@@ -39,5 +39,5 @@
     <!-- 雷达杆的半径和长度 -->
     <xacro:property name="holder_radius" value="0.03" />
-    <xacro:property name="holder_length" value="0.16" />
+    <xacro:property name="holder_length" value="0.10" />
     <!-- 轮胎关节偏移量 -->
     <xacro:property name="wheel_joint_x" value="0.2" />

File: Simulation/gazebo_sim/urdf/robot/robot.urdf.xacro (robot description, xacro)
@@ -30,4 +30,4 @@
     </xacro:VLP-16> -->
     <xacro:include filename="$(find gazebo_sim)/urdf/robot/plugins/gazebo_control_plugin_prefix.xacro" />
-    <xacro:gazebo_control_plugin namespace_prefix="${namespace_prefix}" />
+    <xacro:gazebo_control_plugin/>
 </robot>
