Commit message: delete all ${ns}

File: Simulation/gazebo_sim/urdf/robot/car_base.urdf.xacro (robot description, xacro)
@@ -1,6 +1,6 @@
 <!-- 底盘 -->
 <robot xmlns:xacro="http://www.ros.org/wiki/xacro" name="robot">
-    <link name="${ns}base_footprint" />
-    <link name="${ns}vehicle">
+    <link name="base_footprint" />
+    <link name="vehicle">
         <visual>
             <geometry>
@@ -16,12 +16,12 @@
         <xacro:box_inertial_matrix m="3" l="${car_length}" w="${car_width}" h="${car_height}" />
     </link>
-    <joint name="${ns}vehicle2base_footprint" type="fixed">
-        <parent link="${ns}base_footprint" />
-        <child link="${ns}vehicle" />
+    <joint name="vehicle2base_footprint" type="fixed">
+        <parent link="base_footprint" />
+        <child link="vehicle" />
         <origin xyz="0.0 0.0 ${car_height/2+distance}" />
     </joint>
     <!-- 车轮宏函数 -->
     <xacro:macro name="wheel_func" params="link_name front_flag left_flag">
-        <link name="${ns}${link_name}_wheel">
+        <link name="${link_name}_wheel">
             <visual>
                 <geometry>
@@ -39,7 +39,7 @@
             <xacro:sphere_inertial_matrix m="4" r="${wheel_radius}" />
         </link>
-        <joint name="${ns}${link_name}2vehicle" type="fixed">
-            <parent link="${ns}vehicle" />
-            <child link="${ns}${link_name}_wheel" />
+        <joint name="${link_name}2vehicle" type="fixed">
+            <parent link="vehicle" />
+            <child link="${link_name}_wheel" />
             <origin xyz="${wheel_joint_x* front_flag} ${wheel_joint_y* left_flag} ${wheel_joint_z}" />
             <axis xyz="0.0 1.0 0.0" />
@@ -50,5 +50,5 @@
     <xacro:wheel_func link_name="back_left" front_flag="-1" left_flag="1" />
     <xacro:wheel_func link_name="back_right" front_flag="-1" left_flag="-1" />
-    <link name="${ns}lidar_holder">
+    <link name="lidar_holder">
         <visual>
             <origin xyz="0 0 0" rpy="0 0 0" />
@@ -64,14 +64,14 @@
         <xacro:cylinder_inertial_matrix m="0.1" r="${holder_radius}" h="${holder_length}" />
     </link>
-    <joint name="${ns}lidar_holder2vehicle" type="fixed">
+    <joint name="lidar_holder2vehicle" type="fixed">
         <origin xyz="0.0 0.0 ${car_height/2+holder_length/2}" rpy="0 0 0" />
-        <parent link="${ns}vehicle" />
-        <child link="${ns}lidar_holder" />
+        <parent link="vehicle" />
+        <child link="lidar_holder" />
     </joint>
-    <xacro:gazebo_material ref="${ns}vehicle" color="Red" />
-    <xacro:gazebo_material ref="${ns}lidar_holder" color="Black" />
-    <xacro:gazebo_material ref="${ns}front_left_wheel" color="Black" />
-    <xacro:gazebo_material ref="${ns}front_right_wheel" color="Black" />
-    <xacro:gazebo_material ref="${ns}back_left_wheel" color="Black" />
-    <xacro:gazebo_material ref="${ns}back_right_wheel" color="Black" />
+    <xacro:gazebo_material ref="vehicle" color="Red" />
+    <xacro:gazebo_material ref="lidar_holder" color="Black" />
+    <xacro:gazebo_material ref="front_left_wheel" color="Black" />
+    <xacro:gazebo_material ref="front_right_wheel" color="Black" />
+    <xacro:gazebo_material ref="back_left_wheel" color="Black" />
+    <xacro:gazebo_material ref="back_right_wheel" color="Black" />
 </robot>

File: Simulation/gazebo_sim/urdf/robot/plugins/gazebo_control_plugin.xacro (robot description, xacro)
@@ -3,5 +3,5 @@
     <xacro:macro name="gazebo_control_plugin">
         <!-- mu1静,mu2动，kp 刚度系数 kd 阻尼系数 -->
-        <gazebo reference="${ns}front_left_wheel">
+        <gazebo reference="front_left_wheel">
             <mu1>0.0</mu1>
             <mu2>0.0</mu2>
@@ -11,5 +11,5 @@
             <maxVel>100.0</maxVel>
         </gazebo>
-        <gazebo reference="${ns}front_right_wheel">
+        <gazebo reference="front_right_wheel">
             <mu1>0.0</mu1>
             <mu2>0.0</mu2>
@@ -19,5 +19,5 @@
             <maxVel>100.0</maxVel>
         </gazebo>
-        <gazebo reference="${ns}back_left_wheel">
+        <gazebo reference="back_left_wheel">
             <mu1>0.0</mu1>
             <mu2>0.0</mu2>
@@ -27,5 +27,5 @@
             <maxVel>100.0</maxVel>
         </gazebo>
-        <gazebo reference="${ns}back_right_wheel">
+        <gazebo reference="back_right_wheel">
             <mu1>0.0</mu1>
             <mu2>0.0</mu2>

File: Simulation/gazebo_sim/urdf/robot/robot.urdf.xacro (robot description, xacro)
@@ -8,7 +8,7 @@
     <xacro:include filename="sensor/camera.urdf.xacro" />
     <!-- <xacro:include filename="laser.urdf.xacro" /> -->
-    <joint name="${ns}camera2base_link" type="fixed">
-        <parent link="${ns}vehicle" />
-        <child link="${ns}camera" />
+    <joint name="camera2base_link" type="fixed">
+        <parent link="vehicle" />
+        <child link="camera" />
         <origin xyz="0.2 0 0.12" rpy="0 0 0" />
         <axis xyz="0 0 0" />

File: Simulation/gazebo_sim/urdf/robot/sensor/camera.urdf.xacro (robot description, xacro)
@@ -1,4 +1,4 @@
 <robot xmlns:xacro="http://www.ros.org/wiki/xacro" name="robot">
-  <link name="${ns}camera">
+  <link name="camera">
     <!-- <collision>
       <origin xyz="0 0 0" rpy="0 0 0" />
@@ -19,5 +19,5 @@
     </inertial>
   </link>
-  <gazebo reference="${ns}camera">
+  <gazebo reference="camera">
     <gravity>true</gravity>
     <sensor type="camera" name="camera">

File: Simulation/gazebo_sim/urdf/robot/sensor/laser.urdf.xacro (robot description, xacro)
@@ -1,4 +1,4 @@
 <robot name="laser" xmlns:xacro="http://wiki.ros.org/xacro">
-    <link name="${ns}laser">
+    <link name="laser">
         <visual>
             <origin xyz="0 0 0" rpy="0 0 0" />
@@ -15,12 +15,12 @@
         <xacro:cylinder_inertial_matrix m="0.2" r="${laser_radius}" h="${laser_length}" />
     </link>
-    <joint name="${ns}laser2vehicle" type="fixed">
+    <joint name="laser2vehicle" type="fixed">
         <origin xyz="0.0 -0.2 ${car_height/2+laser_length/2}" rpy="0 -0.0873 ${PI/2}" />
-        <parent link="${ns}vehicle" />
-        <child link="${ns}laser" />
+        <parent link="vehicle" />
+        <child link="laser" />
     </joint>
-    <xacro:gazebo_material ref="${ns}laser" color="Black" />
+    <xacro:gazebo_material ref="laser" color="Black" />
     <!-- laser -->
-    <gazebo reference="${ns}laser">            <!-- get laser's link name -->
+    <gazebo reference="laser">            <!-- get laser's link name -->
         <sensor type="ray" name="rplidar">
             <pose>0 0 0 0 0 0</pose>
@@ -51,5 +51,5 @@
             <plugin name="gazebo_rplidar" filename="libgazebo_ros_laser.so">
                 <topicName>/scan</topicName>
-                <frameName>${ns}laser</frameName>
+                <frameName>laser</frameName>
             </plugin>
         </sensor>

Commit message: add namespace

File: Simulation/gazebo_sim/urdf/robot/car_base.urdf.xacro (robot description, xacro)
@@ -1,6 +1,6 @@
 <!-- 底盘 -->
 <robot xmlns:xacro="http://www.ros.org/wiki/xacro" name="robot">
-    <link name="base_footprint" />
-    <link name="vehicle">
+    <link name="${namespace_prefix}base_footprint" />
+    <link name="${namespace_prefix}vehicle">
         <visual>
             <geometry>
@@ -16,12 +16,12 @@
         <xacro:box_inertial_matrix m="3" l="${car_length}" w="${car_width}" h="${car_height}" />
     </link>
-    <joint name="vehicle2base_footprint" type="fixed">
-        <parent link="base_footprint" />
-        <child link="vehicle" />
+    <joint name="${namespace_prefix}vehicle2base_footprint" type="fixed">
+        <parent link="${namespace_prefix}base_footprint" />
+        <child link="${namespace_prefix}vehicle" />
         <origin xyz="0.0 0.0 ${car_height/2+distance}" />
     </joint>
     <!-- 车轮宏函数 -->
     <xacro:macro name="wheel_func" params="link_name front_flag left_flag">
-        <link name="${link_name}_wheel">
+        <link name="${namespace_prefix}${link_name}_wheel">
             <visual>
                 <geometry>
@@ -39,7 +39,7 @@
             <xacro:sphere_inertial_matrix m="4" r="${wheel_radius}" />
         </link>
-        <joint name="${link_name}2vehicle" type="fixed">
-            <parent link="vehicle" />
-            <child link="${link_name}_wheel" />
+        <joint name="${namespace_prefix}${link_name}2vehicle" type="fixed">
+            <parent link="${namespace_prefix}vehicle" />
+            <child link="${namespace_prefix}${link_name}_wheel" />
             <origin xyz="${wheel_joint_x* front_flag} ${wheel_joint_y* left_flag} ${wheel_joint_z}" />
             <axis xyz="0.0 1.0 0.0" />
@@ -50,5 +50,5 @@
     <xacro:wheel_func link_name="back_left" front_flag="-1" left_flag="1" />
     <xacro:wheel_func link_name="back_right" front_flag="-1" left_flag="-1" />
-    <link name="lidar_holder">
+    <link name="${namespace_prefix}lidar_holder">
         <visual>
             <origin xyz="0 0 0" rpy="0 0 0" />
@@ -64,14 +64,14 @@
         <xacro:cylinder_inertial_matrix m="0.1" r="${holder_radius}" h="${holder_length}" />
     </link>
-    <joint name="lidar_holder2vehicle" type="fixed">
+    <joint name="${namespace_prefix}lidar_holder2vehicle" type="fixed">
         <origin xyz="0.0 0.0 ${car_height/2+holder_length/2}" rpy="0 0 0" />
-        <parent link="vehicle" />
-        <child link="lidar_holder" />
+        <parent link="${namespace_prefix}vehicle" />
+        <child link="${namespace_prefix}lidar_holder" />
     </joint>
-    <xacro:gazebo_material ref="vehicle" color="Red" />
-    <xacro:gazebo_material ref="lidar_holder" color="Black" />
-    <xacro:gazebo_material ref="front_left_wheel" color="Black" />
-    <xacro:gazebo_material ref="front_right_wheel" color="Black" />
-    <xacro:gazebo_material ref="back_left_wheel" color="Black" />
-    <xacro:gazebo_material ref="back_right_wheel" color="Black" />
+    <xacro:gazebo_material ref="${namespace_prefix}vehicle" color="Red" />
+    <xacro:gazebo_material ref="${namespace_prefix}lidar_holder" color="Black" />
+    <xacro:gazebo_material ref="${namespace_prefix}front_left_wheel" color="Black" />
+    <xacro:gazebo_material ref="${namespace_prefix}front_right_wheel" color="Black" />
+    <xacro:gazebo_material ref="${namespace_prefix}back_left_wheel" color="Black" />
+    <xacro:gazebo_material ref="${namespace_prefix}back_right_wheel" color="Black" />
 </robot>

File: Simulation/gazebo_sim/urdf/robot/plugins/gazebo_control_plugin_prefix.xacro (robot description, xacro)
@@ -1,7 +1,8 @@
 <?xml version="1.0"?>
 <robot xmlns:xacro="http://www.ros.org/wiki/xacro">
-    <xacro:macro name="gazebo_control_plugin">
+    <xacro:macro name="gazebo_control_plugin" params="hub_id:=''">
+        <xacro:property name="namespace_prefix" value="${hub_id + '/' if hub_id else ''}" />
         <!-- mu1静,mu2动，kp 刚度系数 kd 阻尼系数 -->
-        <gazebo reference="front_left_wheel">
+        <gazebo reference="${namespace_prefix}front_left_wheel">
             <mu1>0.0</mu1>
             <mu2>0.0</mu2>
@@ -11,5 +12,5 @@
             <maxVel>100.0</maxVel>
         </gazebo>
-        <gazebo reference="front_right_wheel">
+        <gazebo reference="${namespace_prefix}front_right_wheel">
             <mu1>0.0</mu1>
             <mu2>0.0</mu2>
@@ -19,5 +20,5 @@
             <maxVel>100.0</maxVel>
         </gazebo>
-        <gazebo reference="back_left_wheel">
+        <gazebo reference="${namespace_prefix}back_left_wheel">
             <mu1>0.0</mu1>
             <mu2>0.0</mu2>
@@ -27,5 +28,5 @@
             <maxVel>100.0</maxVel>
         </gazebo>
-        <gazebo reference="back_right_wheel">
+        <gazebo reference="${namespace_prefix}back_right_wheel">
             <mu1>0.0</mu1>
             <mu2>0.0</mu2>
@@ -37,8 +38,8 @@
         <gazebo>
             <plugin name="planar_move_controller" filename="libgazebo_ros_planar_move.so">
-                <!-- 里程计和机器人基坐标系（可选，默认已匹配你的配置） -->
-                <odometry_frame>odom</odometry_frame>
-                <robot_base_frame>base_footprint</robot_base_frame>
-                <odometry_topic>odom</odometry_topic>
+                <!-- 里程计和机器人基坐标系，添加命名空间前缀 -->
+                <odometry_frame>${namespace_prefix}odom</odometry_frame>
+                <robot_base_frame>${namespace_prefix}base_footprint</robot_base_frame>
+                <odometry_topic>${namespace_prefix}odom</odometry_topic>
                 <!-- 发布频率（单位Hz） -->
                 <publish_rate>50</publish_rate>

File: Simulation/gazebo_sim/urdf/robot/property.xacro (robot description, xacro)
@@ -1,3 +1,5 @@
 <robot xmlns:xacro="http://www.ros.org/wiki/xacro" name="robot">
+    <xacro:property name="hub_id" value="$(arg hub_id)" />
+    <xacro:property name="namespace_prefix" value="${hub_id + '/' if hub_id else ''}" />
     <xacro:property name="ns" value="$(arg ns)/" />
     <!-- 惯性矩阵 -->

File: Simulation/gazebo_sim/urdf/robot/robot.urdf.xacro (robot description, xacro)
@@ -14,15 +14,15 @@
         <axis xyz="0 0 0" />
     </joint> -->
-    <xacro:VLP-16 parent="lidar_holder" name="velodyne" topic="/velodyne_points" hz="10"
-        min_range="0.55" samples="350" collision_range="0.56" gpu="false"
+    <xacro:VLP-16 namespace_prefix="${namespace_prefix}" parent="lidar_holder"  name="velodyne" topic="velodyne_points" hz="10"
+        min_range="0.55" samples="350" collision_range="0.56" organize_cloud="true" gpu="false"
         min_angle="-3.14159" max_angle="3.14159" vmin_angle="${-7/180*PI}" vmax_angle="${52/180*PI}">
         <origin xyz="0.0 0.0 ${holder_length/2}" rpy="0 0 0" />
     </xacro:VLP-16>
     <!-- <xacro:VLP-16 parent="vehicle" name="velodyne2" topic="/velodyne_points2" hz="10"
-        min_range="0.55" samples="350" collision_range="0.56" gpu="false"
+        min_range="0.55" samples="350" collision_range="0.56" organize_cloud="true" gpu="false"
         min_angle="-3.14159" max_angle="0" vmin_angle="${-7/180*PI}" vmax_angle="${52/180*PI}">
         <origin xyz="0.0 -0.2 ${car_height/2+0.02}" rpy="0 0 0" />
     </xacro:VLP-16> -->
-    <xacro:include filename="$(find gazebo_sim)/urdf/robot/plugins/gazebo_control_plugin.xacro" />
-    <xacro:gazebo_control_plugin />
+    <xacro:include filename="$(find gazebo_sim)/urdf/robot/plugins/gazebo_control_plugin_prefix.xacro" />
+    <xacro:gazebo_control_plugin hub_id="${hub_id}" />
 </robot>

File: Simulation/velodyne_simulator/velodyne_description/urdf/VLP-16.urdf.xacro (robot description, xacro)
@@ -1,58 +1,57 @@
 <?xml version="1.0"?>
 <robot xmlns:xacro="http://www.ros.org/wiki/xacro" name="VLP-16">
-  <xacro:property name="M_PI" value="3.1415926535897931"/>
-  <xacro:macro name="VLP-16" params="*origin parent:=base_link name:=velodyne topic:=/velodyne_points hz:=10 lasers:=16 samples:=1875 collision_range:=0.3 min_range:=0.9 max_range:=130.0 noise:=0.008 min_angle:=-${M_PI} max_angle:=${M_PI} gpu:=false vmin_angle:=-${M_PI} vmax_angle:=${M_PI}">
-    <joint name="${name}_base_mount_joint" type="fixed">
-      <xacro:insert_block name="origin"/>
-      <parent link="${parent}"/>
-      <child link="${name}_base_link"/>
+  <xacro:property name="M_PI" value="3.1415926535897931" />
+  <xacro:macro name="VLP-16"
+    params="*origin namespace_prefix:='' parent:=base_link name:=velodyne organize_cloud:=false topic:=/velodyne_points organize_cloud:=false hz:=10 lasers:=16 samples:=1875 collision_range:=0.5 min_range:=0.6 max_range:=30.0 noise:=0.008 min_angle:=-${M_PI} max_angle:=${M_PI} gpu:=false vmin_angle:=-${M_PI} vmax_angle:=${M_PI}">
+    <joint name="${namespace_prefix}${name}_base_mount_joint" type="fixed">
+      <xacro:insert_block name="origin" />  <!--插入参数宏，对应第一个参数*origin-->
+      <parent link="${namespace_prefix}${parent}" />
+      <child link="${namespace_prefix}${name}_base_link" />
     </joint>
-    <link name="${name}_base_link">
+    <link name="${namespace_prefix}${name}_base_link">
       <inertial>
-        <mass value="0.83"/>
-        <origin xyz="0 0 0.03585"/>
-        <inertia ixx="${(0.83 * (3.0*0.0516*0.0516 + 0.0717*0.0717)) / 12.0}" ixy="0" ixz="0" iyy="${(0.83 * (3.0*0.0516*0.0516 + 0.0717*0.0717)) / 12.0}" iyz="0" izz="${0.5 * 0.83 * (0.0516*0.0516)}"/>
+        <mass value="0.83" />
+        <origin xyz="0 0 0.03585" />
+        <inertia ixx="${(0.83 * (3.0*0.0516*0.0516 + 0.0717*0.0717)) / 12.0}" ixy="0" ixz="0"
+          iyy="${(0.83 * (3.0*0.0516*0.0516 + 0.0717*0.0717)) / 12.0}" iyz="0"
+          izz="${0.5 * 0.83 * (0.0516*0.0516)}" />
       </inertial>
       <visual>
         <geometry>
-          <!-- <mesh filename="package://velodyne_description/meshes/VLP16_base_1.dae"/> -->
-          <mesh filename="file://$(find velodyne_description)/meshes/VLP16_base_1.dae"/>
+          <mesh filename="package://velodyne_description/meshes/VLP16_base_1.dae" />
         </geometry>
       </visual>
       <visual>
         <geometry>
-          <!-- <mesh filename="package://velodyne_description/meshes/VLP16_base_2.dae"/> -->
-          <mesh filename="file://$(find velodyne_description)/meshes/VLP16_base_2.dae"/>
+          <mesh filename="package://velodyne_description/meshes/VLP16_base_2.dae" />
         </geometry>
       </visual>
       <collision>
-        <origin rpy="0 0 0" xyz="0 0 0.03585"/>
+        <origin rpy="0 0 0" xyz="0 0 0.03585" />
         <geometry>
-          <cylinder radius="0.0516" length="0.0717"/>
+          <cylinder radius="0.0516" length="0.0717" />
         </geometry>
       </collision>
     </link>
-    <joint name="${name}_base_scan_joint" type="fixed">
-      <origin xyz="0 0 0.0377" rpy="0 0 0"/>
-      <parent link="${name}_base_link"/>
-      <child link="${name}"/>
+    <joint name="${namespace_prefix}${name}_base_scan_joint" type="fixed">
+      <origin xyz="0 0 0.0377" rpy="0 0 0" />
+      <parent link="${namespace_prefix}${name}_base_link" />
+      <child link="${namespace_prefix}${name}" />
     </joint>
-    <link name="${name}">
+    <link name="${namespace_prefix}${name}">
       <inertial>
-        <mass value="0.01"/>
-        <origin xyz="0 0 0"/>
-        <inertia ixx="1e-7" ixy="0" ixz="0" iyy="1e-7" iyz="0" izz="1e-7"/>
+        <mass value="0.01" />
+        <origin xyz="0 0 0" />
+        <inertia ixx="1e-7" ixy="0" ixz="0" iyy="1e-7" iyz="0" izz="1e-7" />
       </inertial>
       <visual>
-        <origin xyz="0 0 -0.0377"/>
+        <origin xyz="0 0 -0.0377" />
         <geometry>
-          <!-- <mesh filename="package://velodyne_description/meshes/VLP16_scan.dae"/> -->
-          <!-- <mesh $(find velodyne_description)/meshes/VLP16_scan.dae"/> -->
-          <mesh filename="file://$(find velodyne_description)/meshes/VLP16_scan.dae"/>
+          <mesh filename="package://velodyne_description/meshes/VLP16_scan.dae" />
         </geometry>
       </visual>
     </link>
     <!-- Gazebo requires the velodyne_gazebo_plugins package -->
-    <gazebo reference="${name}">
+    <gazebo reference="${namespace_prefix}${name}">
       <xacro:if value="${gpu}">
         <sensor type="gpu_ray" name="${name}-VLP16">
@@ -86,7 +85,8 @@
             </noise>
           </ray>
-          <plugin name="gazebo_ros_laser_controller" filename="libgazebo_ros_velodyne_laser.so">
-            <topicName>${topic}</topicName>
-            <frameName>${name}</frameName>
+          <plugin name="gazebo_ros_laser_controller" filename="libgazebo_ros_velodyne_gpu_laser.so">
+            <topicName>/${namespace_prefix}${topic}</topicName>
+            <frameName>/${namespace_prefix}${name}</frameName>
+            <organize_cloud>${organize_cloud}</organize_cloud>
             <min_range>${min_range}</min_range>
             <max_range>${max_range}</max_range>
@@ -127,6 +127,7 @@
           </ray>
           <plugin name="gazebo_ros_laser_controller" filename="libgazebo_ros_velodyne_laser.so">
-            <topicName>${topic}</topicName>
-            <frameName>${name}</frameName>
+            <topicName>/${namespace_prefix}${topic}</topicName>
+            <frameName>/${namespace_prefix}${name}</frameName>
+            <organize_cloud>${organize_cloud}</organize_cloud>
             <min_range>${min_range}</min_range>
             <max_range>${max_range}</max_range>
