Commit message: error VLP-lidar

File: Simulation/gazebo_sim/urdf/robot/robot.urdf.xacro (robot description, xacro)
@@ -14,11 +14,11 @@
         <axis xyz="0 0 0" />
     </joint> -->
-    <xacro:VLP-16 namespace_prefix="${namespace_prefix}" parent="lidar_holder"  name="velodyne" topic="velodyne_points" hz="10"
-        min_range="0.55" samples="350" collision_range="0.56" organize_cloud="true" gpu="false"
+    <xacro:VLP-16 hub_id="${hub_id}" parent="lidar_holder"  name="velodyne" topic="velodyne_points" hz="10"
+        min_range="0.55" samples="350" collision_range="0.56" gpu="false"
         min_angle="-3.14159" max_angle="3.14159" vmin_angle="${-7/180*PI}" vmax_angle="${52/180*PI}">
         <origin xyz="0.0 0.0 ${holder_length/2}" rpy="0 0 0" />
     </xacro:VLP-16>
     <!-- <xacro:VLP-16 parent="vehicle" name="velodyne2" topic="/velodyne_points2" hz="10"
-        min_range="0.55" samples="350" collision_range="0.56" organize_cloud="true" gpu="false"
+        min_range="0.55" samples="350" collision_range="0.56" gpu="false"
         min_angle="-3.14159" max_angle="0" vmin_angle="${-7/180*PI}" vmax_angle="${52/180*PI}">
         <origin xyz="0.0 -0.2 ${car_height/2+0.02}" rpy="0 0 0" />

File: Simulation/velodyne_simulator/velodyne_description/urdf/VLP-16.urdf.xacro (robot description, xacro)
@@ -3,5 +3,6 @@
   <xacro:property name="M_PI" value="3.1415926535897931" />
   <xacro:macro name="VLP-16"
-    params="*origin namespace_prefix:='' parent:=base_link name:=velodyne organize_cloud:=false topic:=/velodyne_points organize_cloud:=false hz:=10 lasers:=16 samples:=1875 collision_range:=0.5 min_range:=0.6 max_range:=30.0 noise:=0.008 min_angle:=-${M_PI} max_angle:=${M_PI} gpu:=false vmin_angle:=-${M_PI} vmax_angle:=${M_PI}">
+    params="*origin hub_id:='' parent:=base_link name:=velodyne topic:=velodyne_points organize_cloud:=false hz:=10 lasers:=16 samples:=1875 collision_range:=0.5 min_range:=0.6 max_range:=30.0 noise:=0.008 min_angle:=-${M_PI} max_angle:=${M_PI} gpu:=false vmin_angle:=-${M_PI} vmax_angle:=${M_PI}">
+    <xacro:property name="namespace_prefix" value="${hub_id + '/' if hub_id else ''}" />
     <joint name="${namespace_prefix}${name}_base_mount_joint" type="fixed">
       <xacro:insert_block name="origin" />  <!--插入参数宏，对应第一个参数*origin-->
@@ -86,6 +87,6 @@
           </ray>
           <plugin name="gazebo_ros_laser_controller" filename="libgazebo_ros_velodyne_gpu_laser.so">
-            <topicName>/${namespace_prefix}${topic}</topicName>
-            <frameName>/${namespace_prefix}${name}</frameName>
+            <topicName>${namespace_prefix}${topic}</topicName>
+            <frameName>${namespace_prefix}${name}</frameName>
             <organize_cloud>${organize_cloud}</organize_cloud>
             <min_range>${min_range}</min_range>
@@ -127,7 +128,6 @@
           </ray>
           <plugin name="gazebo_ros_laser_controller" filename="libgazebo_ros_velodyne_laser.so">
-            <topicName>/${namespace_prefix}${topic}</topicName>
-            <frameName>/${namespace_prefix}${name}</frameName>
-            <organize_cloud>${organize_cloud}</organize_cloud>
+            <topicName>${namespace_prefix}${topic}</topicName>
+            <frameName>${namespace_prefix}${name}</frameName>
             <min_range>${min_range}</min_range>
             <max_range>${max_range}</max_range>

Commit message: finished gazebo

File: Simulation/gazebo_sim/urdf/robot/robot.urdf.xacro (robot description, xacro)
@@ -19,4 +19,9 @@
         <origin xyz="0.0 0.0 ${holder_length/2}" rpy="0 0 0" />
     </xacro:VLP-16> -->
+    <xacro:VLP-16 parent="denk/lidar_holder"  name="velodyne" topic="denk/velodyne_points" hz="10"
+        min_range="0.55" samples="350" collision_range="0.56" gpu="false"
+        min_angle="-3.14159" max_angle="3.14159" >
+        <origin xyz="0.0 0.0 ${holder_length/2}" rpy="0 0 0" />
+    </xacro:VLP-16>
     <!-- <xacro:VLP-16 parent="vehicle" name="velodyne2" topic="/velodyne_points2" hz="10"
         min_range="0.55" samples="350" collision_range="0.56" gpu="false"

File: Simulation/velodyne_simulator/velodyne_description/urdf/VLP-16.urdf_old.xacro (robot description, xacro)
@@ -1,20 +1,23 @@
 <?xml version="1.0"?>
 <robot xmlns:xacro="http://www.ros.org/wiki/xacro" name="VLP-16">
-  <xacro:property name="M_PI" value="3.1415926535897931"/>
-  <xacro:macro name="VLP-16" params="*origin parent:=base_link name:=velodyne topic:=/velodyne_points hz:=10 lasers:=16 samples:=1875 collision_range:=0.3 min_range:=0.9 max_range:=130.0 noise:=0.008 min_angle:=-${M_PI} max_angle:=${M_PI} gpu:=false">
-    <joint name="${name}_base_mount_joint" type="fixed">
-      <xacro:insert_block name="origin"/>
-      <parent link="${parent}"/>
-      <child link="${name}_base_link"/>
+  <xacro:property name="M_PI" value="3.1415926535897931" />
+  <xacro:macro name="VLP-16"
+    params="*origin hub_id:='' parent:=base_link name:=velodyne topic:=/velodyne_points hz:=10 lasers:=16 samples:=1875 collision_range:=0.5 min_range:=0.6 max_range:=30.0 noise:=0.008 min_angle:=-${M_PI} max_angle:=${M_PI} gpu:=false vmin_angle:=-${M_PI} vmax_angle:=${M_PI}">
+    <xacro:property name="namespace_prefix" value="${hub_id + '/' if hub_id else ''}" />
+    <joint name="${namespace_prefix}${name}_base_mount_joint" type="fixed">
+      <xacro:insert_block name="origin" />  <!--插入参数宏，对应第一个参数*origin-->
+      <parent link="${namespace_prefix}${parent}" />
+      <child link="${namespace_prefix}${name}_base_link" />
     </joint>
-    <link name="${name}_base_link">
+    <link name="${namespace_prefix}${name}_base_link">
       <inertial>
-        <mass value="0.83"/>
-        <origin xyz="0 0 0.03585"/>
-        <inertia ixx="${(0.83 * (3.0*0.0516*0.0516 + 0.0717*0.0717)) / 12.0}" ixy="0" ixz="0" iyy="${(0.83 * (3.0*0.0516*0.0516 + 0.0717*0.0717)) / 12.0}" iyz="0" izz="${0.5 * 0.83 * (0.0516*0.0516)}"/>
+        <mass value="0.83" />
+        <origin xyz="0 0 0.03585" />
+        <inertia ixx="${(0.83 * (3.0*0.0516*0.0516 + 0.0717*0.0717)) / 12.0}" ixy="0" ixz="0"
+          iyy="${(0.83 * (3.0*0.0516*0.0516 + 0.0717*0.0717)) / 12.0}" iyz="0"
+          izz="${0.5 * 0.83 * (0.0516*0.0516)}" />
       </inertial>
       <visual>
         <geometry>
-          <!-- <mesh filename="package://velodyne_description/meshes/VLP16_base_1.dae"/> -->
           <mesh filename="file://$(find velodyne_description)/meshes/VLP16_base_1.dae"/>
         </geometry>
@@ -22,37 +25,34 @@
       <visual>
         <geometry>
-          <!-- <mesh filename="package://velodyne_description/meshes/VLP16_base_2.dae"/> -->
           <mesh filename="file://$(find velodyne_description)/meshes/VLP16_base_2.dae"/>
         </geometry>
       </visual>
       <collision>
-        <origin rpy="0 0 0" xyz="0 0 0.03585"/>
+        <origin rpy="0 0 0" xyz="0 0 0.03585" />
         <geometry>
-          <cylinder radius="0.0516" length="0.0717"/>
+          <cylinder radius="0.0516" length="0.0717" />
         </geometry>
       </collision>
     </link>
-    <joint name="${name}_base_scan_joint" type="fixed">
-      <origin xyz="0 0 0.0377" rpy="0 0 0"/>
-      <parent link="${name}_base_link"/>
-      <child link="${name}"/>
+    <joint name="${namespace_prefix}${name}_base_scan_joint" type="fixed">
+      <origin xyz="0 0 0.0377" rpy="0 0 0" />
+      <parent link="${namespace_prefix}${name}_base_link" />
+      <child link="${namespace_prefix}${name}" />
     </joint>
-    <link name="${name}">
+    <link name="${namespace_prefix}${name}">
       <inertial>
-        <mass value="0.01"/>
-        <origin xyz="0 0 0"/>
-        <inertia ixx="1e-7" ixy="0" ixz="0" iyy="1e-7" iyz="0" izz="1e-7"/>
+        <mass value="0.01" />
+        <origin xyz="0 0 0" />
+        <inertia ixx="1e-7" ixy="0" ixz="0" iyy="1e-7" iyz="0" izz="1e-7" />
       </inertial>
       <visual>
-        <origin xyz="0 0 -0.0377"/>
+        <origin xyz="0 0 -0.0377" />
         <geometry>
-          <!-- <mesh filename="package://velodyne_description/meshes/VLP16_scan.dae"/> -->
-          <!-- <mesh $(find velodyne_description)/meshes/VLP16_scan.dae"/> -->
-          <mesh filename="file://$(find velodyne_description)/meshes/VLP16_scan.dae"/>
+          <mesh filename="package://velodyne_description/meshes/VLP16_scan.dae" />
         </geometry>
       </visual>
     </link>
     <!-- Gazebo requires the velodyne_gazebo_plugins package -->
-    <gazebo reference="${name}">
+    <gazebo reference="${namespace_prefix}${name}">
       <xacro:if value="${gpu}">
         <sensor type="gpu_ray" name="${name}-VLP16">
@@ -71,7 +71,6 @@
                 <samples>${lasers}</samples>
                 <resolution>1</resolution>
-                <min_angle>-${15.0*M_PI/180.0}</min_angle>
-                <max_angle>
-                  ${15.0*M_PI/180.0}</max_angle>
+                <min_angle>${vmin_angle}</min_angle>
+                <max_angle>${vmax_angle}</max_angle>
               </vertical>
             </scan>
@@ -87,7 +86,7 @@
             </noise>
           </ray>
-          <plugin name="gazebo_ros_laser_controller" filename="libgazebo_ros_velodyne_laser.so">
-            <topicName>${topic}</topicName>
-            <frameName>${name}</frameName>
+          <plugin name="gazebo_ros_laser_controller" filename="libgazebo_ros_velodyne_gpu_laser.so">
+            <topicName>${namespace_prefix}${topic}</topicName>
+            <frameName>${namespace_prefix}${name}</frameName>
             <min_range>${min_range}</min_range>
             <max_range>${max_range}</max_range>
@@ -112,7 +111,6 @@
                 <samples>${lasers}</samples>
                 <resolution>1</resolution>
-                <min_angle>-${15.0*M_PI/180.0}</min_angle>
-                <max_angle>
-                  ${15.0*M_PI/180.0}</max_angle>
+                <min_angle>${vmin_angle}</min_angle>
+                <max_angle>${vmax_angle}</max_angle>
               </vertical>
             </scan>
@@ -129,6 +127,6 @@
           </ray>
           <plugin name="gazebo_ros_laser_controller" filename="libgazebo_ros_velodyne_laser.so">
-            <topicName>${topic}</topicName>
-            <frameName>${name}</frameName>
+            <topicName>${namespace_prefix}${topic}</topicName>
+            <frameName>${namespace_prefix}${name}</frameName>
             <min_range>${min_range}</min_range>
             <max_range>${max_range}</max_range>
